Commit message: add controller

File: src/abot_description/urdf/abot.xacro (robot description, xacro)
@@ -8,5 +8,7 @@
 	<!-- Matherials -->
 	<xacro:include filename="$(find abot_description)/urdf/abot_materials.xacro" />
-	<!-- abot_base -->
+	<!-- clearance -->
+  <xacro:property name="clearance" value="0.018" />
+  <!-- abot_base -->
   <link
     name="abot_base">
@@ -61,4 +63,19 @@
 	<child link="abot_base" />
 </joint>
+<!-- base_footprint -->
+<link name="base_footprint">
+	<visual>
+		<origin xyz="0 0 0" rpy="0 0 0" />
+		<geometry>
+			<cylinder length="0.001" radius="0.010" />
+		</geometry>
+		<material name="Blue" />
+	</visual>
+</link>
+<joint name="base_footprint_to_base_link" type="fixed">
+	<origin xyz="0 0 ${clearance}" rpy="0 0 0" />
+	<parent link="base_footprint" />
+	<child link="base_link" />
+</joint>
 <!-- Wheels -->
 <xacro:include filename="$(find abot_description)/urdf/abot_left_wheel.xacro" />

Commit message: add robot_base

File: src/abot_description/urdf/abot.xacro (robot description, xacro)
@@ -8,6 +8,10 @@
 	<!-- Matherials -->
 	<xacro:include filename="$(find abot_description)/urdf/abot_materials.xacro" />
-	<!-- clearance -->
+	<!-- parameters -->
   <xacro:property name="clearance" value="0.018" />
+  <xacro:property name="wheel_radius" value="0.0325"/>
+  <xacro:property name="wheel_separation" value="0.128"/>
+  <xacro:property name="wheel_width" value="0.026"/>
+  <xacro:property name="PI" value="3.1415926"/>
   <!-- abot_base -->
   <link

File: src/abot_description/urdf/abot_left_wheel.xacro (robot description, xacro)
@@ -54,3 +54,29 @@
       xyz="0 0 1" />
   </joint>
+  <link name="left_wheel">
+	<visual>
+		<origin xyz="0 0 0" rpy="${PI/2} 0 0" />
+		<geometry>
+			<cylinder length="${wheel_width}" radius="${wheel_radius}"/>
+		</geometry>
+		<material name="Green" />
+	</visual>
+	<collision>
+		<origin xyz="0 0 0" rpy="${PI/2} 0 0" />
+		<geometry>
+			<cylinder length="${wheel_width}" radius="${wheel_radius}"/>
+		</geometry>
+	</collision>
+</link>
+<joint name="left_wheel_to_abot_left_wheel" type="fixed">
+	<origin xyz="0 0 0" rpy="0 0 0" />
+	<parent link="left_wheel" />
+	<child link="abot_left_wheel" />
+</joint>
+<joint name="left_wheel_to_base" type="continuous">
+	<origin xyz="0 0.068 0.0145" rpy="0 0 0" />
+	<parent link="abot_base" />
+	<child link="left_wheel" />
+	<axis xyz="0 1 0" />
+</joint>
 </robot>

File: src/abot_description/urdf/abot_right_wheel.xacro (robot description, xacro)
@@ -54,3 +54,29 @@
       xyz="0 0 1" />
   </joint>
+  <link name="right_wheel">
+	<visual>
+		<origin xyz="0 0 0" rpy="${PI/2} 0 0" />
+		<geometry>
+			<cylinder length="${wheel_width}" radius="${wheel_radius}"/>
+		</geometry>
+		<material name="Green" />
+	</visual>
+	<collision>
+		<origin xyz="0 0 0" rpy="${PI/2} 0 0" />
+		<geometry>
+			<cylinder length="${wheel_width}" radius="${wheel_radius}"/>
+		</geometry>
+	</collision>
+</link>
+<joint name="right_wheel_to_abot_right_wheel" type="fixed">
+	<origin xyz="0 0 0" rpy="0 0 0" />
+	<parent link="right_wheel" />
+	<child link="abot_right_wheel" />
+</joint>
+<joint name="right_wheel_to_base" type="continuous">
+	<origin xyz="0 -0.068 0.0145" rpy="0 0 0" />
+	<parent link="abot_base" />
+	<child link="right_wheel" />
+	<axis xyz="0 1 0" />
+</joint>
 </robot>

Commit message: edit model xacro

File: src/abot_description/urdf/abot.xacro (robot description, xacro)
@@ -19,5 +19,5 @@
     <inertial>
       <origin
-        xyz="0 0.00150000000000001 1.38777878078145E-17"
+        xyz="3.52930394689292E-18 4.62395285906123E-18 0.0015"
         rpy="0 0 0" />
       <mass
@@ -72,5 +72,5 @@
 		<origin xyz="0 0 0" rpy="0 0 0" />
 		<geometry>
-			<cylinder length="0.001" radius="0.010" />
+			<cylinder length="0.001" radius="0.100" />
 		</geometry>
 		<material name="Blue" />
@@ -85,3 +85,5 @@
 <xacro:include filename="$(find abot_description)/urdf/abot_left_wheel.xacro" />
 <xacro:include filename="$(find abot_description)/urdf/abot_right_wheel.xacro" />
+<!-- Sensors -->
+<xacro:include filename="$(find abot_description)/urdf/abot_sensors.xacro" />
 </robot>

File: src/abot_description/urdf/abot_left_wheel.xacro (robot description, xacro)
@@ -41,17 +41,4 @@
     </collision>
   </link>
-  <joint
-    name="left_wheel_to_base"
-    type="continuous">
-    <origin
-      xyz="-0.04 0.003 0.05"
-      rpy="0 0 0" />
-    <parent
-      link="abot_base" />
-    <child
-      link="abot_left_wheel" />
-    <axis
-      xyz="0 0 1" />
-  </joint>
   <link name="left_wheel">
 	<visual>
@@ -75,5 +62,5 @@
 </joint>
 <joint name="left_wheel_to_base" type="continuous">
-	<origin xyz="0 0.068 0.0145" rpy="0 0 0" />
+	<origin xyz="0.04 0.0625 0.00299999999999998" rpy="0 0 0" />
 	<parent link="abot_base" />
 	<child link="left_wheel" />

File: src/abot_description/urdf/abot_right_wheel.xacro (robot description, xacro)
@@ -41,17 +41,4 @@
     </collision>
   </link>
-  <joint
-    name="right_wheel_to_base"
-    type="continuous">
-    <origin
-      xyz="-0.04 0.003 -0.075"
-      rpy="0 0 0" />
-    <parent
-      link="abot_base" />
-    <child
-      link="abot_right_wheel" />
-    <axis
-      xyz="0 0 1" />
-  </joint>
   <link name="right_wheel">
 	<visual>
@@ -75,5 +62,5 @@
 </joint>
 <joint name="right_wheel_to_base" type="continuous">
-	<origin xyz="0 -0.068 0.0145" rpy="0 0 0" />
+	<origin xyz="0.04 -0.0625 0.00300000000000001" rpy="0 0 0" />
 	<parent link="abot_base" />
 	<child link="right_wheel" />

Commit message: wheel separetion

File: src/abot_description/urdf/abot.xacro (robot description, xacro)
@@ -11,5 +11,5 @@
   <xacro:property name="clearance" value="0.018" />
   <xacro:property name="wheel_radius" value="0.0325"/>
-  <xacro:property name="wheel_separation" value="0.128"/>
+  <xacro:property name="wheel_separation" value="0.135"/>
   <xacro:property name="wheel_width" value="0.026"/>
   <xacro:property name="PI" value="3.1415926"/>
