Commit message: set equal robot and rviz rotation by right position wheels from base

File: src/abot_description/urdf/abot_left_wheel.xacro (robot description, xacro)
@@ -62,5 +62,5 @@
 </joint>
 <joint name="left_wheel_to_base" type="continuous">
-	<origin xyz="0.04 0.0625 0.00299999999999998" rpy="0 0 0" />
+	<origin xyz="0.04 0.0638 0.00299999999999998" rpy="0 0 0" />
 	<parent link="abot_base" />
 	<child link="left_wheel" />

File: src/abot_description/urdf/abot_right_wheel.xacro (robot description, xacro)
@@ -62,5 +62,5 @@
 </joint>
 <joint name="right_wheel_to_base" type="continuous">
-	<origin xyz="0.04 -0.0625 0.00300000000000001" rpy="0 0 0" />
+	<origin xyz="0.04 -0.0638 0.00300000000000001" rpy="0 0 0" />
 	<parent link="abot_base" />
 	<child link="right_wheel" />
